Commit message: Add Tkinter open/close GUI and gripper fixes
- Add robotiq_2f_gripper_gui.py and robotiq_2f_85_gui.launch
- Update gripper driver, modbus RTU, action client example
- Update 2F-85 visualization launch and xacro

File: robotiq_2f_85_gripper_visualization/urdf/robotiq_arg2f_85_model.xacro (robot description, xacro)
@@ -3,3 +3,26 @@
   <xacro:include filename="$(find robotiq_2f_85_gripper_visualization)/urdf/robotiq_arg2f_85_model_macro.xacro" />
   <xacro:robotiq_arg2f_85 prefix=""/>
+  <link name="robotiq_gripper_coupling">
+    <visual>
+      <geometry>
+        <mesh
+          filename="package://robotiq_2f_85_gripper_visualization/meshes/visual/robotiq_gripper_coupling.stl"
+          scale="0.001 0.001 0.001"/>
+      </geometry>
+      <material name="">
+        <color rgba="0.13 0.13 0.13 1" />
+      </material>
+    </visual>
+    <collision>
+      <origin xyz="0 0 0.0065" rpy="0 0 0" />
+      <geometry>
+        <cylinder radius="0.038" length="0.018" />
+      </geometry>
+    </collision>
+  </link>
+  <joint name="gripper_base_to_coupling" type="fixed">
+    <parent link="robotiq_arg2f_base_link"/>
+    <child link="robotiq_gripper_coupling"/>
+    <origin xyz="0 0 0" rpy="0 0 3.14"/>
+  </joint>
 </robot>
